Commit message: adaptive transmission is what's effing up

File: robot/ur5_soma.urdf.xacro (robot description, xacro)
@@ -7,14 +7,45 @@
   <xacro:include filename="$(find ur_description)/urdf/ur5.urdf.xacro" />
   <xacro:include filename="$(find ur_description)/urdf/common.gazebo.xacro" />
+  <xacro:include filename="$(find soma_ur5)/robot/ee_attachments.xacro" />
   <!-- arm -->
-  <xacro:ur5_robot prefix="ur5_arm/" joint_limited="true"/>
+  <xacro:ur5_robot prefix="" joint_limited="true"/>
   <link name="world" />
   <joint name="world_joint" type="fixed">
     <parent link="world" />
-    <child link = "ur5_arm/base_link" />
+    <child link = "base_link" />
     <origin xyz="0.0 0.0 0.0" rpy="0.0 0.0 0.0" />
   </joint>
-  <xacro:include filename="$(find soma_ur5)/robot/ee_attachments.xacro" />
-  <xacro:wrist_sensor parent="ur5_arm/base_link" child="ati_base_measurement"/> <!--tool0 -->
+  <xacro:wrist_sensor parent="tool0" child="ati_base_measurement"/> <!--tool0 -->
+<joint name="merdose_joint" type="fixed">
+        <origin xyz="0 0 0.01" rpy="0 0 0"/>
+      <parent link="ati_base_measurement"/>
+      <child link="merdose"/>
+      <!--limit lower="-0.00001" upper="0.00001" effort="100" velocity="100"/>
+      <axis xyz="0 0 1" /-->
+    </joint>
+    <link name="merdose">
+      <inertial>
+        <mass value="0.255"/>
+        <origin xyz="0 0 0.0"  />
+        <xacro:cylinder_inertia_def radius="0.0177" length="0.2" mass="0.255"/>
+      </inertial>
+      <visual>
+        <!-- origin xyz="0 0 0.00725" rpy="0 0 0"/ -->
+        <origin xyz="0 0.0 0" rpy="0 0 0"/>
+        <geometry>
+          <cylinder radius="0.0177" length="0.2"/>
+          <!--mesh filename="package://force_torque_sensor/model/meshes/ati_gamma.stl"/-->
+        </geometry>
+         <material name="green">
+          <color rgba="0 .8 0 1"/>
+         </material>
+      </visual>
+      <collision>
+        <origin xyz="0 0 0.0" rpy="0 0 0"/>
+        <geometry>
+          <cylinder radius="0.0177" length="0.2"/>
+        </geometry>
+      </collision>
+    </link>
   <!--xacro:ft_sensor parent="tool0" name="wrist" type="ati_gamma">
     <origin xyz="0 0 0.0165" rpy="0 0 0"/>
@@ -27,7 +58,7 @@
     <axis xyz="0 0 1" />
   </joint-->
-  <!--xacro:soft_hand parent="ati_base_measurement" name="soft_hand" left="true" withAdaptiveTransmission="false" useMimicTag="false">
-    <origin xyz="0 0 0.0" rpy="0 0 0"/>
-  </xacro:soft_hand-->
+  <xacro:soft_hand parent="merdose" name="soft_hand" left="true" withAdaptiveTransmission="true" useMimicTag="true">
+    <origin xyz="0 0 0.1" rpy="0 0 0"/>
+  </xacro:soft_hand>
  <!-- Frame coincident with all-zeros TCP on UR controller -->
     <!--link name="hand_attachment">
