Commit message: Aleluia

File: robot/ee_attachments.xacro (robot description, xacro)
@@ -90,4 +90,5 @@
 </gazebo>
   <transmission name="sensor_trans">
+        <robotNamespace>ati</robotNamespace>
       <type>transmission_interface/SimpleTransmission</type>
       <joint name="wrist_sensor_joint">

File: robot/ur5_soma.urdf.xacro (robot description, xacro)
@@ -1,8 +1,7 @@
 <?xml version="1.0"?>
 <robot xmlns:xacro="http://www.ros.org/wiki/xacro"
-       name="ur5_soma">
+       name="soft_hand">
   <xacro:include filename="$(find soft_hand_description)/model/soft_hand.urdf.xacro"/>
   <xacro:include filename="$(find force_torque_sensor)/model/ft_sensor.urdf.xacro"/>
-  <!-- ur5 -->
   <xacro:include filename="$(find ur_description)/urdf/ur5.urdf.xacro" />
   <xacro:include filename="$(find ur_description)/urdf/common.gazebo.xacro" />
@@ -16,11 +15,9 @@
     <origin xyz="0.0 0.0 0.0" rpy="0.0 0.0 0.0" />
   </joint>
-  <xacro:wrist_sensor parent="tool0" child="ati_base_measurement"/> <!--tool0 -->
-<joint name="merdose_joint" type="fixed">
+  <xacro:wrist_sensor parent="tool0" child="ati_base_measurement"/>
+<!--joint name="merdose_joint" type="fixed">
         <origin xyz="0 0 0.01" rpy="0 0 0"/>
       <parent link="ati_base_measurement"/>
       <child link="merdose"/>
-      <!--limit lower="-0.00001" upper="0.00001" effort="100" velocity="100"/>
-      <axis xyz="0 0 1" /-->
     </joint>
     <link name="merdose">
@@ -31,9 +28,7 @@
       </inertial>
       <visual>
-        <!-- origin xyz="0 0 0.00725" rpy="0 0 0"/ -->
         <origin xyz="0 0.0 0" rpy="0 0 0"/>
         <geometry>
           <cylinder radius="0.0177" length="0.2"/>
-          <!--mesh filename="package://force_torque_sensor/model/meshes/ati_gamma.stl"/-->
         </geometry>
          <material name="green">
@@ -47,5 +42,5 @@
         </geometry>
       </collision>
-    </link>
+    </link-->
   <!--xacro:ft_sensor parent="tool0" name="wrist" type="ati_gamma">
     <origin xyz="0 0 0.0165" rpy="0 0 0"/>
@@ -58,6 +53,27 @@
     <axis xyz="0 0 1" />
   </joint-->
-  <xacro:soft_hand parent="merdose" name="soft_hand" left="true" withAdaptiveTransmission="true" useMimicTag="true">
-    <origin xyz="0 0 0.1" rpy="0 0 0"/>
+  <!--link name="box">
+    <inertial>
+      <mass value="50.0"/>
+      <inertia  ixx="1" ixy="0.00"  ixz="0.00" iyy="1" iyz="0.00" izz="1" />
+    </inertial>
+    <visual>
+      <origin xyz="0 0 0.50" rpy="0 0 0"/>
+      <geometry>
+        <box size="1.0 1.0 1.0"/>
+      </geometry>
+    </visual>
+    <collision>
+      <origin xyz="0 0 0.50" rpy="0 0 0"/>
+      <geometry>
+        <box size="1.0 1.0 1.0"/>
+      </geometry>
+    </collision>
+  </link>
+  <gazebo reference="box">
+    <static>true</static>
+  </gazebo-->
+  <xacro:soft_hand parent="ati_base_measurement" name="soft_hand"  withAdaptiveTransmission="true" useMimicTag="false" left="false">
+    <origin xyz="0 0 0.01" rpy="0 0 0"/>
   </xacro:soft_hand>
  <!-- Frame coincident with all-zeros TCP on UR controller -->

Commit message: Simulator working

File: robot/ee_attachments.xacro (robot description, xacro)
@@ -89,5 +89,5 @@
 </plugin>
 </gazebo>
-  <transmission name="sensor_trans">
+  <!--transmission name="sensor_trans">
         <robotNamespace>ati</robotNamespace>
       <type>transmission_interface/SimpleTransmission</type>
@@ -98,5 +98,5 @@
         <mechanicalReduction>1</mechanicalReduction>
       </actuator>
-    </transmission>
+    </transmission-->
 	</xacro:macro>
 </robot>

File: robot/ur5_soma.urdf.xacro (robot description, xacro)
@@ -16,73 +16,6 @@
   </joint>
   <xacro:wrist_sensor parent="tool0" child="ati_base_measurement"/>
-<!--joint name="merdose_joint" type="fixed">
-        <origin xyz="0 0 0.01" rpy="0 0 0"/>
-      <parent link="ati_base_measurement"/>
-      <child link="merdose"/>
-    </joint>
-    <link name="merdose">
-      <inertial>
-        <mass value="0.255"/>
-        <origin xyz="0 0 0.0"  />
-        <xacro:cylinder_inertia_def radius="0.0177" length="0.2" mass="0.255"/>
-      </inertial>
-      <visual>
-        <origin xyz="0 0.0 0" rpy="0 0 0"/>
-        <geometry>
-          <cylinder radius="0.0177" length="0.2"/>
-        </geometry>
-         <material name="green">
-          <color rgba="0 .8 0 1"/>
-         </material>
-      </visual>
-      <collision>
-        <origin xyz="0 0 0.0" rpy="0 0 0"/>
-        <geometry>
-          <cylinder radius="0.0177" length="0.2"/>
-        </geometry>
-      </collision>
-    </link-->
-  <!--xacro:ft_sensor parent="tool0" name="wrist" type="ati_gamma">
-    <origin xyz="0 0 0.0165" rpy="0 0 0"/>
-  </xacro:ft_sensor-->
-  <!--joint name="hand_attachment_joint" type="revolute">
-    <parent link="wrist_ati_gamma_measure" />
-    <child link = "hand_attachment" />
-    <origin xyz="0.0 0.0 0.0" rpy="0.0 0.0 0.0" />
-    <limit lower="-0.00001" upper="0.00001" effort="100" velocity="100"/>
-    <axis xyz="0 0 1" />
-  </joint-->
-  <!--link name="box">
-    <inertial>
-      <mass value="50.0"/>
-      <inertia  ixx="1" ixy="0.00"  ixz="0.00" iyy="1" iyz="0.00" izz="1" />
-    </inertial>
-    <visual>
-      <origin xyz="0 0 0.50" rpy="0 0 0"/>
-      <geometry>
-        <box size="1.0 1.0 1.0"/>
-      </geometry>
-    </visual>
-    <collision>
-      <origin xyz="0 0 0.50" rpy="0 0 0"/>
-      <geometry>
-        <box size="1.0 1.0 1.0"/>
-      </geometry>
-    </collision>
-  </link>
-  <gazebo reference="box">
-    <static>true</static>
-  </gazebo-->
   <xacro:soft_hand parent="ati_base_measurement" name="soft_hand"  withAdaptiveTransmission="true" useMimicTag="false" left="false">
     <origin xyz="0 0 0.01" rpy="0 0 0"/>
   </xacro:soft_hand>
- <!-- Frame coincident with all-zeros TCP on UR controller -->
-    <!--link name="hand_attachment">
-      <collision>
-        <geometry>
-          <box size="0.01 0.01 0.01"/>
-        </geometry>
-        <origin rpy="0 0 0" xyz="0.01 0 0"/>
-      </collision>
-    </link-->
 </robot>

Commit message: Remapping topics for sim/real coherence

File: robot/ee_attachments.xacro (robot description, xacro)
@@ -17,5 +17,5 @@
 	<xacro:macro name="wrist_sensor" params="parent child">
 		<joint name="wrist_joint" type="fixed">
-		    <origin xyz="0 0 0.01" rpy="0 0 0"/>
+		    <origin xyz="0 0 0.01" rpy="0 0 ${pi/2}"/>
 			<parent link="${parent}"/>
 			<child link="ati_base"/>
@@ -85,5 +85,5 @@
 <plugin name="ft_sensor" filename="libgazebo_ros_ft_sensor.so">
 <updateRate>100.0</updateRate>
-<topicName>ft_sensor_topic</topicName>
+<topicName>netft_data_sim</topicName>
 <jointName>wrist_sensor_joint</jointName>
 </plugin>

File: robot/ur5_soma.urdf.xacro (robot description, xacro)
@@ -16,5 +16,5 @@
   </joint>
   <xacro:wrist_sensor parent="tool0" child="ati_base_measurement"/>
-  <xacro:soft_hand parent="ati_base_measurement" name="soft_hand"  withAdaptiveTransmission="true" useMimicTag="false" left="false">
+  <xacro:soft_hand parent="ati_base_measurement" name="soft_hand"  withAdaptiveTransmission="true" useMimicTag="false" left="true">
     <origin xyz="0 0 0.01" rpy="0 0 0"/>
   </xacro:soft_hand>

Commit message: new setup

File: robot/ee_attachments.xacro (robot description, xacro)
@@ -15,7 +15,7 @@
 			 ixy="0" iyz="0" ixz="0"/>
 	</xacro:macro>
-	<xacro:macro name="wrist_sensor" params="parent child">
+	<xacro:macro name="wrist_sensor" params="parent child rot">
 		<joint name="wrist_joint" type="fixed">
-		    <origin xyz="0 0 0.01" rpy="0 0 ${pi/2}"/>
+		    <origin xyz="0 0 0.01" rpy="0 0 ${rot}"/>
 			<parent link="${parent}"/>
 			<child link="ati_base"/>

File: robot/ur5_soma.urdf.xacro (robot description, xacro)
@@ -15,5 +15,5 @@
     <origin xyz="0.0 0.0 0.0" rpy="0.0 0.0 0.0" />
   </joint>
-  <xacro:wrist_sensor parent="tool0" child="ati_base_measurement"/>
+  <xacro:wrist_sensor parent="tool0" child="ati_base_measurement" rot="${3*pi/4}"/>
   <xacro:soft_hand parent="ati_base_measurement" name="soft_hand"  withAdaptiveTransmission="true" useMimicTag="false" left="true">
     <origin xyz="0 0 0.01" rpy="0 0 0"/>
